Commit message: Move lidar position

File: interbotix_ros_xslocobots/interbotix_xslocobot_descriptions/urdf/lidar.urdf.xacro (robot description, xacro)
@@ -34,6 +34,6 @@
     </gazebo>
     <joint name="lidar" type="fixed">
-      <origin rpy="0 0 ${pi}" xyz="0 0 0.09425"/>
-      <parent link="$(arg robot_name)/lidar_tower_link"/>
+      <origin rpy="0 0 0" xyz="-0.09277 0 0.25"/>
+      <parent link="$(arg robot_name)/base_footprint"/>
       <child link="$(arg robot_name)/laser_frame_link"/>
     </joint>
